File: PCBs/hall_ring/Hall_ring.sch (KiCad schematic (older format))
At the start: 19 parts, among them J1 Conn_02x05_Odd_Even, J2 Conn_01x03_Female, U1 DRV5053_LPG, U2 DRV5053_LPG, U3 DRV5053_LPG, U4 DRV5053_LPG, U5 DRV5053_LPG, U6 DRV5053_LPG, U7 DRV5053_LPG

Commit message: added makaniu BMS board V2, and wayfinders 6cell BMS.
Parts:
- D1: symbol Custom:LED_RG -> Hall_ring-rescue:LED_RG-Custom
- U1, U2, U3, U4, U5, U6, U7: symbol Custom:DRV5053_LPG -> Hall_ring-rescue:DRV5053_LPG-Custom
Changed lines of the file:
@@
 $EndDescr
 $Comp
-L Custom:DRV5053_LPG U3
+L Hall_ring-rescue:DRV5053_LPG-Custom U3
 U 1 1 5F033524
 P 3600 1350
@@
 $EndComp
 $Comp
-L Custom:DRV5053_LPG U4
+L Hall_ring-rescue:DRV5053_LPG-Custom U4
 U 1 1 5F035BFA
 P 4950 1350
@@
 $EndComp
 $Comp
-L Custom:DRV5053_LPG U6
+L Hall_ring-rescue:DRV5053_LPG-Custom U6
 U 1 1 5F0383D1
 P 7650 1350
@@
 $EndComp
 $Comp
-L Custom:DRV5053_LPG U5
+L Hall_ring-rescue:DRV5053_LPG-Custom U5
 U 1 1 5F0370E1
 P 6300 1350
@@
 	1500 3600 1600 3600
 $Comp
-L Custom:DRV5053_LPG U7
+L Hall_ring-rescue:DRV5053_LPG-Custom U7
 U 1 1 5F07B9E2
 P 1200 4000
@@
 $EndComp
 $Comp
-L Custom:DRV5053_LPG U1
+L Hall_ring-rescue:DRV5053_LPG-Custom U1
 U 1 1 5EF55C80
 P 900 1350
@@
 $EndComp
 $Comp
-L Custom:DRV5053_LPG U2
+L Hall_ring-rescue:DRV5053_LPG-Custom U2
 U 1 1 5F065A9F
 P 2250 1350
@@
 	9550 2700 9250 2700
 $Comp
-L Custom:LED_RG D1
+L Hall_ring-rescue:LED_RG-Custom D1
 U 1 1 5F0AA8C7
 P 6450 3150

Commit message: updates to battery managemennt wayfinder boards, and makaniu hall sensor ring and BMS
Parts:
- C1, C2, C3, C4, C5, C6, C7: footprint Capacitor_SMD:C_0603_1608Metric_Pad1.05x0.95mm_HandSolder -> Capacitor_SMD:C_0402_1005Metric; Digikey (none) -> 1276-1043-2-ND
- D1: Digikey (none) -> 160-1939-ND
- J1: Digikey (none) -> H125941-ND
- J2: Digikey (none) -> 455-1705-ND
- R1: footprint Resistor_SMD:R_0603_1608Metric_Pad1.05x0.95mm_HandSolder -> Resistor_SMD:R_0402_1005Metric; Digikey (none) -> YAG5286TR-ND
- R2: footprint Resistor_SMD:R_0603_1608Metric_Pad1.05x0.95mm_HandSolder -> Resistor_SMD:R_0402_1005Metric; Digikey (none) -> 311-200LRTR-ND
- U1, U2, U3, U4, U5, U6, U7: Digikey (none) -> 296-DRV5032DULPGMCT-ND
Connections:
- wire segments 60 -> 63
Changed lines of the file:
@@
 F 2 "Package_TO_SOT_THT:TO-92Flat" H 3600 1350 50  0001 C CNN
 F 3 "" H 3600 1350 50  0001 C CNN
+F 4 "296-DRV5032DULPGMCT-ND" H 3600 1350 50  0001 C CNN "Digikey"
 	1    3600 1350
 	1    0    0    1
@@
 F 2 "Package_TO_SOT_THT:TO-92Flat" H 4950 1350 50  0001 C CNN
 F 3 "" H 4950 1350 50  0001 C CNN
+F 4 "296-DRV5032DULPGMCT-ND" H 4950 1350 50  0001 C CNN "Digikey"
 	1    4950 1350
 	1    0    0    1
@@
 F 2 "Package_TO_SOT_THT:TO-92Flat" H 7650 1350 50  0001 C CNN
 F 3 "" H 7650 1350 50  0001 C CNN
+F 4 "296-DRV5032DULPGMCT-ND" H 7650 1350 50  0001 C CNN "Digikey"
 	1    7650 1350
 	1    0    0    1
@@
 F 2 "Package_TO_SOT_THT:TO-92Flat" H 6300 1350 50  0001 C CNN
 F 3 "" H 6300 1350 50  0001 C CNN
+F 4 "296-DRV5032DULPGMCT-ND" H 6300 1350 50  0001 C CNN "Digikey"
 	1    6300 1350
 	1    0    0    1
@@
 Wire Wire Line
 	9550 2250 9550 2400
-Text Notes 950  2700 0    50   ~ 0
+Text Notes 1250 1850 0    50   ~ 0
 6 hall sensors are connected to an 8 pin connector that leads to the Pi\n
 Text Notes 1000 4350 0    50   ~ 0
@@
 F 0 "C3" H 4265 996 50  0000 L CNN
 F 1 "0.1uF" H 4265 905 50  0000 L CNN
-F 2 "Capacitor_SMD:C_0603_1608Metric_Pad1.05x0.95mm_HandSolder" H 4188 800 50  0001 C CNN
+F 2 "Capacitor_SMD:C_0402_1005Metric" H 4188 800 50  0001 C CNN
 F 3 "~" H 4150 950 50  0001 C CNN
+F 4 "1276-1043-2-ND" H 4150 950 50  0001 C CNN "Digikey"
 	1    4150 950
 	1    0    0    -1
@@
 F 0 "C4" H 5615 996 50  0000 L CNN
 F 1 "0.1uF" H 5615 905 50  0000 L CNN
-F 2 "Capacitor_SMD:C_0603_1608Metric_Pad1.05x0.95mm_HandSolder" H 5538 800 50  0001 C CNN
+F 2 "Capacitor_SMD:C_0402_1005Metric" H 5538 800 50  0001 C CNN
 F 3 "~" H 5500 950 50  0001 C CNN
+F 4 "1276-1043-2-ND" H 5500 950 50  0001 C CNN "Digikey"
 	1    5500 950
 	1    0    0    -1
@@
 F 0 "C5" H 6965 996 50  0000 L CNN
 F 1 "0.1uF" H 6965 905 50  0000 L CNN
-F 2 "Capacitor_SMD:C_0603_1608Metric_Pad1.05x0.95mm_HandSolder" H 6888 800 50  0001 C CNN
+F 2 "Capacitor_SMD:C_0402_1005Metric" H 6888 800 50  0001 C CNN
 F 3 "~" H 6850 950 50  0001 C CNN
+F 4 "1276-1043-2-ND" H 6850 950 50  0001 C CNN "Digikey"
 	1    6850 950
 	1    0    0    -1
@@
 F 0 "C6" H 8315 996 50  0000 L CNN
 F 1 "0.1uF" H 8315 905 50  0000 L CNN
-F 2 "Capacitor_SMD:C_0603_1608Metric_Pad1.05x0.95mm_HandSolder" H 8238 800 50  0001 C CNN
+F 2 "Capacitor_SMD:C_0402_1005Metric" H 8238 800 50  0001 C CNN
 F 3 "~" H 8200 950 50  0001 C CNN
+F 4 "1276-1043-2-ND" H 8200 950 50  0001 C CNN "Digikey"
 	1    8200 950
 	1    0    0    -1
@@
 	1600 3600 1600 3450
 Wire Wire Line
-	1750 3750 2350 3750
+	1750 3750 1950 3750
 Connection ~ 1750 3750
 Wire Wire Line
@@
 F 0 "C7" H 1865 3646 50  0000 L CNN
 F 1 "0.1uF" H 1865 3555 50  0000 L CNN
-F 2 "Capacitor_SMD:C_0603_1608Metric_Pad1.05x0.95mm_HandSolder" H 1788 3450 50  0001 C CNN
+F 2 "Capacitor_SMD:C_0402_1005Metric" H 1788 3450 50  0001 C CNN
 F 3 "~" H 1750 3600 50  0001 C CNN
+F 4 "1276-1043-2-ND" H 1750 3600 50  0001 C CNN "Digikey"
 	1    1750 3600
 	1    0    0    -1
@@
 F 2 "Connector_JST:JST_PH_B3B-PH-K_1x03_P2.00mm_Vertical" H 2550 3750 50  0001 C CNN
 F 3 "~" H 2550 3750 50  0001 C CNN
+F 4 "455-1705-ND" H 2550 3750 50  0001 C CNN "Digikey"
 	1    2550 3750
 	1    0    0    -1
@@
 F 2 "Package_TO_SOT_THT:TO-92Flat" H 1200 4000 50  0001 C CNN
 F 3 "" H 1200 4000 50  0001 C CNN
+F 4 "296-DRV5032DULPGMCT-ND" H 1200 4000 50  0001 C CNN "Digikey"
 	1    1200 4000
 	1    0    0    1
@@
 Wire Wire Line
 	2350 3850 2150 3850
-Wire Wire Line
-	2150 3850 2150 3900
-Wire Wire Line
-	2150 3900 1500 3900
 $Comp
 L Device:R R1
@@
 F 0 "R1" V 7693 3250 50  0000 C CNN
 F 1 "300" V 7784 3250 50  0000 C CNN
-F 2 "Resistor_SMD:R_0603_1608Metric_Pad1.05x0.95mm_HandSolder" V 7830 3250 50  0001 C CNN
+F 2 "Resistor_SMD:R_0402_1005Metric" V 7830 3250 50  0001 C CNN
 F 3 "~" H 7900 3250 50  0001 C CNN
+F 4 "YAG5286TR-ND" H 7900 3250 50  0001 C CNN "Digikey"
 	1    7900 3250
 	0    1    1    0
@@
 F 0 "R2" V 7693 3650 50  0000 C CNN
 F 1 "200" V 7784 3650 50  0000 C CNN
-F 2 "Resistor_SMD:R_0603_1608Metric_Pad1.05x0.95mm_HandSolder" V 7830 3650 50  0001 C CNN
+F 2 "Resistor_SMD:R_0402_1005Metric" V 7830 3650 50  0001 C CNN
 F 3 "~" H 7900 3650 50  0001 C CNN
+F 4 "311-200LRTR-ND" H 7900 3650 50  0001 C CNN "Digikey"
 	1    7900 3650
 	0    1    1    0
@@
 F 0 "C1" H 1565 996 50  0000 L CNN
 F 1 "0.1uF" H 1565 905 50  0000 L CNN
-F 2 "Capacitor_SMD:C_0603_1608Metric_Pad1.05x0.95mm_HandSolder" H 1488 800 50  0001 C CNN
+F 2 "Capacitor_SMD:C_0402_1005Metric" H 1488 800 50  0001 C CNN
 F 3 "~" H 1450 950 50  0001 C CNN
+F 4 "1276-1043-2-ND" H 1450 950 50  0001 C CNN "Digikey"
 	1    1450 950
 	1    0    0    -1
@@
 F 2 "Package_TO_SOT_THT:TO-92Flat" H 900 1350 50  0001 C CNN
 F 3 "" H 900 1350 50  0001 C CNN
+F 4 "296-DRV5032DULPGMCT-ND" H 900 1350 50  0001 C CNN "Digikey"
 	1    900  1350
 	1    0    0    1
@@
 F 0 "C2" H 2915 996 50  0000 L CNN
 F 1 "0.1uF" H 2915 905 50  0000 L CNN
-F 2 "Capacitor_SMD:C_0603_1608Metric_Pad1.05x0.95mm_HandSolder" H 2838 800 50  0001 C CNN
+F 2 "Capacitor_SMD:C_0402_1005Metric" H 2838 800 50  0001 C CNN
 F 3 "~" H 2800 950 50  0001 C CNN
+F 4 "1276-1043-2-ND" H 2800 950 50  0001 C CNN "Digikey"
 	1    2800 950
 	1    0    0    -1
@@
 F 2 "Package_TO_SOT_THT:TO-92Flat" H 2250 1350 50  0001 C CNN
 F 3 "" H 2250 1350 50  0001 C CNN
+F 4 "296-DRV5032DULPGMCT-ND" H 2250 1350 50  0001 C CNN "Digikey"
 	1    2250 1350
 	1    0    0    1
@@
 F 2 "Connector_Hirose:Hirose_DF11-10DP-2DSA_2x05_P2.00mm_Vertical" H 8950 2600 50  0001 C CNN
 F 3 "~" H 8950 2600 50  0001 C CNN
+F 4 "H125941-ND" H 8950 2600 50  0001 C CNN "Digikey"
 	1    8950 2600
 	1    0    0    -1
@@
 F 2 "Connector_PinHeader_2.00mm:PinHeader_1x03_P2.00mm_Vertical" H 6450 3150 50  0001 C CNN
 F 3 "" H 6450 3150 50  0001 C CNN
+F 4 "160-1939-ND" H 6450 3150 50  0001 C CNN "Digikey"
 	1    6450 3150
 	1    0    0    -1
 $EndComp
+$Comp
+L power:GND #PWR0101
+U 1 1 5F95140C
+P 1950 3750
+F 0 "#PWR0101" H 1950 3500 50  0001 C CNN
+F 1 "GND" H 1955 3577 50  0000 C CNN
+F 2 "" H 1950 3750 50  0001 C CNN
+F 3 "" H 1950 3750 50  0001 C CNN
+	1    1950 3750
+	1    0    0    -1
+$EndComp
+Connection ~ 1950 3750
+Wire Wire Line
+	1950 3750 2350 3750
+Wire Wire Line
+	2150 4000 1600 4000
+Wire Wire Line
+	1600 4000 1600 3900
+Wire Wire Line
+	1600 3900 1500 3900
+Wire Wire Line
+	2150 3850 2150 4000
 $EndSCHEMATC
