File: PCBs/endcap/Maka Niu Endcap.sch (EAGLE design)
At the start: 70 parts, among them J1 U.FL, J2 KELLER_BREAKOUT, J3 GPS_PROG, Q1 20V/0.2A/8MHz/1.2Ω/1Vth, Q2 20V/0.2A/8MHz/1.2Ω/1Vth, U1 P9221-R03MM_PAD, U2 XM1110 GPS, U3 ICM-20948, U4 1.8V/100mA

Commit message: Add files via upload
Finalized for production
Parts:
- renumbered U$3 to COIL
Changed lines of the file:
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@@
 <attribute name="MP" value="0877591450"/>
 </part>
-<part name="U$3" library="maka-niu" deviceset="CHARGING_COIL" device=""/>
+<part name="COIL" library="maka-niu" deviceset="CHARGING_COIL" device=""/>
 <part name="GND1" library="supply1" library_urn="urn:adsk.eagle:library:371" deviceset="GND" device=""/>
 <part name="C10" library="maka-niu" deviceset="C0603" device="C0603W" value="10uF">
@@
 <attribute name="DIGI-KEY_PART_NUMBER" value="732-7556-1-ND"/>
 <attribute name="MF" value="Würth Elektronik"/>
-<attribute name="MP" value="885012205061
-"/>
+<attribute name="MP" value="885012205061 "/>
 </part>
 <part name="C5" library="rcl" library_urn="urn:adsk.eagle:library:334" deviceset="C-EU" device="C0402" package3d_urn="urn:adsk.eagle:package:23626/2" value="22nF/50V">
@@
 <attribute name="DIGI-KEY_PART_NUMBER" x="30.48" y="101.6" size="1.27" layer="96" display="off"/>
 </instance>
-<instance part="U$3" gate="G$1" x="-12.7" y="66.04" smashed="yes">
+<instance part="COIL" gate="G$1" x="-12.7" y="66.04" smashed="yes">
 <attribute name="NAME" x="-11.43" y="68.58" size="1.778" layer="95" font="vector"/>
 <attribute name="VALUE" x="-11.43" y="63.5" size="1.778" layer="96" font="vector" align="top-left"/>
@@
 <pinref part="U1" gate="Q$1" pin="AC2"/>
 <wire x1="45.72" y1="55.88" x2="43.18" y2="55.88" width="0.1524" layer="91"/>
-<pinref part="U$3" gate="G$1" pin="2"/>
+<pinref part="COIL" gate="G$1" pin="2"/>
 <wire x1="43.18" y1="55.88" x2="27.94" y2="55.88" width="0.1524" layer="91"/>
 <wire x1="27.94" y1="55.88" x2="17.78" y2="55.88" width="0.1524" layer="91"/>
@@
 <net name="LC" class="0">
 <segment>
-<pinref part="U$3" gate="G$1" pin="1"/>
+<pinref part="COIL" gate="G$1" pin="1"/>
 <wire x1="-7.62" y1="76.2" x2="-12.7" y2="76.2" width="0.1524" layer="91"/>
 <wire x1="-12.7" y1="76.2" x2="-12.7" y2="71.12" width="0.1524" layer="91"/>
