File: PCBs/battery_manager/Maka_BMS.sch (KiCad schematic (older format))
At the start: 83 parts, among them J8 T1M-10-F-SH-L-K, J9 Molex 087340-1424, Q1 FDC645N, Q2 FDC645N, Q3 FDC645N, Q4 Si3483CDV, Q5 Si3483CDV, Q6 FDC645N, U1 AP63205, U2 TPS70933DBV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

Commit message: Icreased trace thickness and rerouted higher freq and power paths in the battery management board
Parts:
- C24: value 1.75uF -> 0.15uF
Changed lines of the file:
@@
 encoding utf-8
 Sheet 1 1
-Title "Makaniu Simple BMS"
-Date ""
-Rev "000x4"
+Title "Makaniu BMS"
+Date "2020-08-13"
+Rev "0"
 Comp "Open Ocean Initiative"
-Comment1 "Drawn By:Lui Kawasumi"
+Comment1 "Drawn By: Lui Kawasumi"
 Comment2 ""
 Comment3 ""
 Comment4 ""
 $EndDescr
-Wire Wire Line
-	9500 5250 9200 5250
 Wire Wire Line
 	4900 2000 4900 2050
@@
 Text GLabel 9400 5450 0    50   Output ~ 0
 GPS_INT
-Text GLabel 9200 5250 0    50   Input ~ 0
-~TS_EOC~
 Text GLabel 10350 5250 2    50   Output ~ 0
 ~INT~
@@
 P 6650 1500
 F 0 "C24" V 6700 1300 50  0000 R CNN
-F 1 "1.75uF" V 6600 1300 50  0000 R CNN
+F 1 "0.15uF" V 6600 1300 50  0000 R CNN
 F 2 "Capacitor_SMD:C_0402_1005Metric" H 6688 1350 50  0001 C CNN
 F 3 "~" H 6650 1500 50  0001 C CNN
@@
 $EndComp
 Connection ~ 7250 1350
+Wire Wire Line
+	9500 5250 9200 5250
+Text GLabel 9200 5250 0    50   Input ~ 0
+~TS_EOC~
 $EndSCHEMATC

Commit message: changed current sensing resistor values on the BMS board to appropriately trip short and over current situations, adn to appropriately end incomig charge
Parts:
- R29: value 0.033 -> 0.06
- R31: value 0.025 -> 0.1
- R8: value 0.001 -> 0.02
Changed lines of the file:
@@
 P 2150 3650
 F 0 "R8" V 2050 3650 50  0000 C CNN
-F 1 "0.001" V 2150 3650 50  0000 C CNN
+F 1 "0.02" V 2150 3650 50  0000 C CNN
 F 2 "Resistor_SMD:R_1206_3216Metric_Pad1.42x1.75mm_HandSolder" V 2080 3650 50  0001 C CNN
 F 3 "~" H 2150 3650 50  0001 C CNN
@@
 P 10650 2750
 F 0 "R31" V 10550 2750 50  0000 C CNN
-F 1 "0.025" V 10650 2750 50  0000 C CNN
+F 1 "0.1" V 10650 2750 50  0000 C CNN
 F 2 "Resistor_SMD:R_1206_3216Metric_Pad1.42x1.75mm_HandSolder" V 10580 2750 50  0001 C CNN
 F 3 "~" H 10650 2750 50  0001 C CNN
@@
 P 9250 2200
 F 0 "R29" V 9150 2200 50  0000 C CNN
-F 1 "0.033" V 9250 2200 50  0000 C CNN
+F 1 "0.06" V 9250 2200 50  0000 C CNN
 F 2 "Resistor_SMD:R_1206_3216Metric_Pad1.42x1.75mm_HandSolder" V 9180 2200 50  0001 C CNN
 F 3 "~" H 9250 2200 50  0001 C CNN

Commit message: assigned digikey part to every item in battery management schematic, and created BOM
Parts:
- 11.1: Digikey (none) -> 36-241-ND
- 3.4_1: value 3.4- -> 3.4; Digikey (none) -> 36-240-ND
- 3.4_2: value 3.4+ -> 3.4; Digikey (none) -> 36-241-ND
- C1, C13, C15, C16: Digikey (none) -> 490-7202-1-ND
- C10: Digikey (none) -> 1276-6836-1-ND
- C14: Digikey (none) -> 1276-1900-1-ND
- C17: Digikey (none) -> 490-12269-1-ND
- C18: value 0.1Uf -> 0.1uF; Digikey (none) -> 732-7495-1-ND
- C19: value 0.12uF -> 0.22uF; Digikey (none) -> 490-12265-1-ND
- C2, C3, C4, C5: Digikey (none) -> 732-7495-1-ND
- C20: Digikey (none) -> 311-1713-1-ND
- C21: Digikey (none) -> 311-1039-1-ND
- C22, C23: value 20uF -> 22uF; Digikey (none) -> 1276-7076-1-ND
- C24: value 0.15uF -> 0.22uF; Digikey (none) -> 490-12265-1-ND
- C6, C8, C9: Digikey (none) -> 490-10017-1-ND
- C7: Digikey (none) -> 490-13234-1-ND
- D1, D2: Digikey (none) -> BAS5202VH6327XTSA1CT-ND
- D3, D4: Digikey (none) -> CRS08QMCT-ND
- J8: Digikey (none) -> SAM11993-ND
- J9: Digikey (none) -> 23-0873401424-ND
- L1: Digikey (none) -> 490-10651-1-ND
- L2, L3: Digikey (none) -> 541-1093-2-ND
- Q1, Q2, Q3, Q6: Digikey (none) -> FDC645NCT-ND
- Q4, Q5: Digikey (none) -> SI3483CDV-T1-GE3CT-ND
- R1, R13, R2, R3, R4, R5, R6: Digikey (none) -> YAG1234CT-ND
- R10: value 4.5K -> 10K; Digikey (none) -> 311-10.0KLRCT-ND
- R11, R12, R14: Digikey (none) -> 311-1.00MLRCT-ND
- R15, R17: Digikey (none) -> 311-10.0KLRCT-ND
- R16, R23: Digikey (none) -> 311-100KLRCT-ND
- R18: value 450K -> 470K; Digikey (none) -> 311-470KJRCT-ND
- R19: value 250K -> 270K; Digikey (none) -> 311-270KJRCT-ND
- R20: Digikey (none) -> YAG5696CT-ND
- R21: value 47K -> 0
- R22: Digikey (none) -> YAG3119CT-ND
- R24: Digikey (none) -> YAG3108CT-ND
- R25: Digikey (none) -> YAG2293CT-ND
- R26, R27: Digikey (none) -> 311-3.01KLRCT-ND
- R28: Digikey (none) -> YAG1447CT-ND
- R29: Digikey (none) -> WSLC-.06CT-ND
- R30: Digikey (none) -> YAG3081CT-ND
- R31: Digikey (none) -> 311-0.1ANCT-ND
- R32: value 13.3K -> 10.7k; Digikey (none) -> 311-10.7KLRCT-ND
- R33: value 150K -> 120k; Digikey (none) -> 311-120KJRCT-ND
- R8: Digikey (none) -> WSLP-.02CT-ND
- TH1, TH2: Digikey (none) -> P12985CT-ND
- U1: Digikey (none) -> AP63205WU-7DICT-ND
- U2: Digikey (none) -> 296-35483-1-ND
- U3: Digikey (none) -> 296-50995-1-ND
- U4: Digikey (none) -> LTC6994CS6-1#TRMPBFCT-ND
- U5: Digikey (none) -> LTC4007EGN#PBF-ND
- U6: Digikey (none) -> LMR62014XMF/NOPBCT-ND

Commit message: completed the wireless charger PCB design as rev 0. bom is compiled
Parts:
- J8: symbol Custom:T1M-10-F-SH-L-K -> Maka_BMS-rescue:T1M-10-F-SH-L-K-Custom
- U1: symbol Custom:AP63205 -> Maka_BMS-rescue:AP63205-Custom
- U2: symbol Custom:TPS70933DBV -> Maka_BMS-rescue:TPS70933DBV-Custom
- U3: symbol Custom:BQ77915 -> Maka_BMS-rescue:BQ77915-Custom
Other:
- note added: "C22 wrongly routed"
- note added: "WRONG!, make C13 a 100nF\n"
Changed lines of the file:
@@
 	4900 1800 3750 1800
 $Comp
-L Custom:BQ77915 U3
+L Maka_BMS-rescue:BQ77915-Custom U3
 U 1 1 5F22EDFB
 P 3150 1200
@@
 ~DELAYED_OFF~
 $Comp
-L Custom:AP63205 U1
+L Maka_BMS-rescue:AP63205-Custom U1
 U 1 1 5FD494D7
 P 2250 5200
@@
 	8450 1950 8850 1950
 $Comp
-L Custom:T1M-10-F-SH-L-K J8
+L Maka_BMS-rescue:T1M-10-F-SH-L-K-Custom J8
 U 1 1 5F28B09D
 P 6700 5650
@@
 NoConn ~ 10000 5550
 $Comp
-L Custom:TPS70933DBV U2
+L Maka_BMS-rescue:TPS70933DBV-Custom U2
 U 1 1 5FAD69CC
 P 2250 6050
@@
 $EndComp
 $Comp
-L Custom:+CHARGE #PWR0104
+L Maka_BMS-rescue:+CHARGE-Custom #PWR0104
 U 1 1 5FA19A89
 P 10150 2200
@@
 $EndComp
 $Comp
-L Custom:+CHARGE #PWR0105
+L Maka_BMS-rescue:+CHARGE-Custom #PWR0105
 U 1 1 5FA1A2D1
 P 750 4700
@@
 Text GLabel 9200 5250 0    50   Input ~ 0
 ~TS_EOC~
+Text Notes 2200 4850 0    79   ~ 0
+WRONG!, make C13 a 100nF\n
+Text Notes 9750 1850 0    79   ~ 0
+C22 wrongly routed
 $EndSCHEMATC

Commit message: added makaniu BMS board V2, and wayfinders 6cell BMS.
Parts:
- C1, C14, C15, C16, C22, C23: footprint Capacitor_SMD:C_0603_1608Metric_Pad1.05x0.95mm_HandSolder -> Capacitor_SMD:C_0603_1608Metric
- C13: value 10uF -> 0.1uF; footprint Capacitor_SMD:C_0603_1608Metric_Pad1.05x0.95mm_HandSolder -> Capacitor_SMD:C_0603_1608Metric; Digikey 490-7202-1-ND -> 732-7495-1-ND
Connections:
- wire segments 299 -> 300
Other:
- note removed: "C22 wrongly routed"
- note removed: "WRONG!, make C13 a 100nF\n"
Changed lines of the file:
@@
 Wire Notes Line
 	5350 4300 5350 550
-Wire Wire Line
-	10150 2350 10150 2200
 $Comp
 L power:Earth #PWR037
@@
 F 0 "C16" H 3885 5604 50  0000 R CNN
 F 1 "10uF" H 3885 5695 50  0000 R CNN
-F 2 "Capacitor_SMD:C_0603_1608Metric_Pad1.05x0.95mm_HandSolder" H 4038 5500 50  0001 C CNN
+F 2 "Capacitor_SMD:C_0603_1608Metric" H 4038 5500 50  0001 C CNN
 F 3 "~" H 4000 5650 50  0001 C CNN
 F 4 "490-7202-1-ND" H 4000 5650 50  0001 C CNN "Digikey"
@@
 F 0 "C15" H 3485 5604 50  0000 R CNN
 F 1 "10uF" H 3485 5695 50  0000 R CNN
-F 2 "Capacitor_SMD:C_0603_1608Metric_Pad1.05x0.95mm_HandSolder" H 3638 5500 50  0001 C CNN
+F 2 "Capacitor_SMD:C_0603_1608Metric" H 3638 5500 50  0001 C CNN
 F 3 "~" H 3600 5650 50  0001 C CNN
 F 4 "490-7202-1-ND" H 3600 5650 50  0001 C CNN "Digikey"
@@
 P 2750 5350
 F 0 "C13" H 2635 5304 50  0000 R CNN
-F 1 "10uF" H 2635 5395 50  0000 R CNN
-F 2 "Capacitor_SMD:C_0603_1608Metric_Pad1.05x0.95mm_HandSolder" H 2788 5200 50  0001 C CNN
+F 1 "0.1uF" H 2635 5395 50  0000 R CNN
+F 2 "Capacitor_SMD:C_0603_1608Metric" H 2788 5200 50  0001 C CNN
 F 3 "~" H 2750 5350 50  0001 C CNN
-F 4 "490-7202-1-ND" H 2750 5350 50  0001 C CNN "Digikey"
+F 4 "732-7495-1-ND" H 2750 5350 50  0001 C CNN "Digikey"
 	1    2750 5350
 	-1   0    0    1
@@
 F 0 "C1" H 1035 5754 50  0000 R CNN
 F 1 "10uF" H 1035 5845 50  0000 R CNN
-F 2 "Capacitor_SMD:C_0603_1608Metric_Pad1.05x0.95mm_HandSolder" H 1188 5650 50  0001 C CNN
+F 2 "Capacitor_SMD:C_0603_1608Metric" H 1188 5650 50  0001 C CNN
 F 3 "~" H 1150 5800 50  0001 C CNN
 F 4 "490-7202-1-ND" H 1150 5800 50  0001 C CNN "Digikey"
@@
 F 0 "C14" H 2735 6404 50  0000 R CNN
 F 1 "4.7uF" H 2735 6495 50  0000 R CNN
-F 2 "Capacitor_SMD:C_0603_1608Metric_Pad1.05x0.95mm_HandSolder" H 2888 6300 50  0001 C CNN
+F 2 "Capacitor_SMD:C_0603_1608Metric" H 2888 6300 50  0001 C CNN
 F 3 "~" H 2850 6450 50  0001 C CNN
 F 4 "	1276-1900-1-ND" H 2850 6450 50  0001 C CNN "Digikey"
@@
 $EndComp
 Wire Wire Line
-	9850 2350 10150 2350
-Connection ~ 9850 2350
-Wire Wire Line
 	7450 2650 6600 2650
 Wire Wire Line
@@
 Wire Wire Line
 	8950 3700 8950 3750
-Wire Wire Line
-	9550 3150 9850 3150
 Connection ~ 9550 3150
 $Comp
@@
 F 0 "C23" H 10685 3554 50  0000 R CNN
 F 1 "22uF" H 10685 3645 50  0000 R CNN
-F 2 "Capacitor_SMD:C_0603_1608Metric_Pad1.05x0.95mm_HandSolder" H 10838 3450 50  0001 C CNN
+F 2 "Capacitor_SMD:C_0603_1608Metric" H 10838 3450 50  0001 C CNN
 F 3 "~" H 10800 3600 50  0001 C CNN
 F 4 "1276-7076-1-ND" H 10800 3600 50  0001 C CNN "Digikey"
@@
 	9850 2750 9900 2750
 Wire Wire Line
-	9850 2750 9850 2650
-Wire Wire Line
 	8450 2450 8450 2550
-$Comp
-L Device:C C22
-U 1 1 5F68A573
-P 9850 2500
-F 0 "C22" H 9735 2454 50  0000 R CNN
-F 1 "22uF" H 9735 2545 50  0000 R CNN
-F 2 "Capacitor_SMD:C_0603_1608Metric_Pad1.05x0.95mm_HandSolder" H 9888 2350 50  0001 C CNN
-F 3 "~" H 9850 2500 50  0001 C CNN
-F 4 "1276-7076-1-ND" H 9850 2500 50  0001 C CNN "Digikey"
-	1    9850 2500
-	-1   0    0    1
-$EndComp
 Wire Wire Line
 	8600 2050 8800 2050
@@
 	8600 2350 9250 2350
 Connection ~ 9250 2350
-Wire Wire Line
-	9250 2350 9850 2350
 $Comp
 L Device:R R29
@@
 U 1 1 5F690C9E
 P 9150 2550
-F 0 "Q5" H 9355 2504 50  0000 L CNN
-F 1 "Si3483CDV" H 9355 2595 50  0000 L CNN
+F 0 "Q5" H 9350 2600 50  0000 L CNN
+F 1 "Si3483CDV" H 9350 2700 50  0000 L CNN
 F 2 "Custom:SOT-23-6_mosfet" H 9350 2650 50  0001 C CNN
 F 3 "~" H 9150 2550 50  0001 C CNN
@@
 Text GLabel 9200 5250 0    50   Input ~ 0
 ~TS_EOC~
-Text Notes 2200 4850 0    79   ~ 0
-WRONG!, make C13 a 100nF\n
-Text Notes 9750 1850 0    79   ~ 0
-C22 wrongly routed
+Wire Wire Line
+	9550 3150 9850 3150
+Wire Wire Line
+	9850 2750 9850 2650
+$Comp
+L Device:C C22
+U 1 1 5F68A573
+P 9650 2350
+F 0 "C22" H 9535 2304 50  0000 R CNN
+F 1 "22uF" H 9535 2395 50  0000 R CNN
+F 2 "Capacitor_SMD:C_0603_1608Metric" H 9688 2200 50  0001 C CNN
+F 3 "~" H 9650 2350 50  0001 C CNN
+F 4 "1276-7076-1-ND" H 9650 2350 50  0001 C CNN "Digikey"
+	1    9650 2350
+	-1   0    0    1
+$EndComp
+$Comp
+L power:Earth #PWR?
+U 1 1 67887441
+P 9650 2500
+F 0 "#PWR?" H 9650 2250 50  0001 C CNN
+F 1 "Earth" H 9650 2350 50  0001 C CNN
+F 2 "" H 9650 2500 50  0001 C CNN
+F 3 "~" H 9650 2500 50  0001 C CNN
+	1    9650 2500
+	1    0    0    -1
+$EndComp
+Wire Wire Line
+	9250 2350 9500 2350
+Wire Wire Line
+	9500 2350 9500 2200
+Wire Wire Line
+	9500 2200 9650 2200
+Connection ~ 9650 2200
+Wire Wire Line
+	9650 2200 10150 2200
 $EndSCHEMATC

Commit message: updates to battery managemennt wayfinder boards, and makaniu hall sensor ring and BMS
Parts:
- removed 3.4_2: 3.4, Custom:TruHole_Batter_Contact_Pad_with_9mm_clear, symbol Connector_Generic:Conn_01x01
- removed C24: 0.22uF, Capacitor_SMD:C_0402_1005Metric, symbol Device:C
- removed D1: BAS5202VH6327, Diode_SMD:D_0402_1005Metric, symbol Device:D
- removed D4: CRS08, Diode_SMD:D_SOD-123, symbol Device:D
- removed R33: 120k, Resistor_SMD:R_0402_1005Metric, symbol Device:R
- removed U6: LMR62014XMF, Package_TO_SOT_SMD:SOT-23-5, symbol Regulator_Switching:LMR62014XMF
- added 7.4_2: 7.4, Custom:TruHole_Batter_Contact_Pad_with_9mm_clear, symbol Connector_Generic:Conn_01x01
- added C11: 10uF, Capacitor_SMD:C_0603_1608Metric, symbol Device:C
- added C12: 15nF, Capacitor_SMD:C_0402_1005Metric, symbol Device:C
- added D1: 30V 5A, Diode_SMD:D_SMA, symbol Device:D_Schottky
- added D4: 60V 3A, Custom:D_SOD-123EP, symbol Device:D_Schottky
- added R7: 100K, Resistor_SMD:R_0402_1005Metric, symbol Device:R
- added R9: 15K, Resistor_SMD:R_0402_1005Metric, symbol Device:R
- added U6: MP3213, Package_SO:MSOP-8-1EP_3x3mm_P0.65mm_EP1.95x2.15mm, symbol Custom:MP3213
- 0.0: renamed from 0_1; value 0 -> 0.0; footprint TestPoint:TestPoint_THTPad_D1.5mm_Drill0.7mm -> Custom:TruHole_Batter_Contact_Pad_with_9mm_clear; Digikey (none) -> 36-240-ND
- 11.1: footprint Custom:TruHole_Batter_Contact_Pad_with_9mm_clear -> TestPoint:TestPoint_THTPad_D1.5mm_Drill0.7mm; Digikey 36-241-ND -> (none)
- 3.4: renamed from 3.4_1; footprint Custom:TruHole_Batter_Contact_Pad_with_9mm_clear -> TestPoint:TestPoint_THTPad_D1.5mm_Drill0.7mm; Digikey 36-240-ND -> (none)
- 7.4_1: renamed from 7.4; footprint TestPoint:TestPoint_THTPad_D1.5mm_Drill0.7mm -> Custom:TruHole_Batter_Contact_Pad_with_9mm_clear; Digikey (none) -> 36-241-ND
- C1, C15, C16: LCSC (none) -> C96446; RemQ (none) -> 3
- C10: value 4.7uF -> 1nF; Digikey 1276-6836-1-ND -> 478-1101-2-ND; LCSC (none) -> C1523; RemQ (none) -> 0
- C13: footprint Capacitor_SMD:C_0603_1608Metric -> Capacitor_SMD:C_0402_1005Metric; LCSC (none) -> C155422; RemQ (none) -> 3
- C17: LCSC (none) -> C47339; RemQ (none) -> 0
- C18, C2, C3, C4, C5: LCSC (none) -> C155422; RemQ (none) -> 3
- C19: LCSC (none) -> C16772; RemQ (none) -> 0
- C21: LCSC (none) -> C1538; RemQ (none) -> 0
- C6, C8, C9: LCSC (none) -> C52923; RemQ (none) -> 1
- C7: value 2.2uF -> 10uF; footprint Capacitor_SMD:C_0402_1005Metric -> Capacitor_SMD:C_0603_1608Metric; Digikey 490-13234-1-ND -> 490-7202-1-ND; LCSC (none) -> C96446; RemQ (none) -> 3
- D2: value BAS5202VH6327 -> 30V 5A; footprint Diode_SMD:D_0402_1005Metric -> Diode_SMD:D_SMA; symbol Device:D -> Device:D_Schottky; Digikey BAS5202VH6327XTSA1CT-ND -> SK56A-LTPMSTR-ND
- J8: value T1M-10-F-SH-L-K -> ‎SAM16035-ND‎
- L2, L3: Digikey 541-1093-2-ND -> 541-1093-1-ND
- R1, R13, R2, R3, R4, R5, R6: LCSC (none) -> C11702; RemQ (none) -> 5
- R10, R15, R17: LCSC (none) -> C25744; RemQ (none) -> 2
- R11, R12, R14: LCSC (none) -> C26083; RemQ (none) -> 2
- R16, R23: LCSC (none) -> C25741; RemQ (none) -> 0
- R21: value 0 -> 110K; Digikey (none) -> ‎311-110KLRCT-ND
- R22: LCSC (none) -> C13187; RemQ (none) -> 0
- R24: LCSC (none) -> C122546; RemQ (none) -> 0
- R25: LCSC (none) -> C17765; RemQ (none) -> 0
- R26, R27: LCSC (none) -> C25889; RemQ (none) -> 0
- R28: LCSC (none) -> C25903; RemQ (none) -> 0
- R30: LCSC (none) -> C25876; RemQ (none) -> 0
- R31: LCSC (none) -> C25334; RemQ (none) -> 0
- R32: value 10.7k -> 10K; Digikey 311-10.7KLRCT-ND -> 311-10.0KLRCT-ND; LCSC (none) -> C25744; RemQ (none) -> 2
- TH1: Digikey P12985CT-ND -> 495-5814-1-ND
- TH2: value 10K -> DNP; Digikey P12985CT-ND -> 495-5814-1-ND
Connections:
- net labels added: BATT_OUT, GND_OUT
- net labels removed: +CHARGE
- wire segments 300 -> 304
Other:
- moved on the sheet: J8

Commit message: Minor notes on BMS pcb project
Other:
- note added: "CUT THIS LINE"
Changed lines of the file:
@@
 Text Label 950  5400 0    79   ~ 0
 BATT_OUT
+Wire Notes Line
+	6250 2350 7350 2350
+Wire Notes Line
+	7350 2350 7350 1950
+Wire Notes Line
+	7350 1950 6250 1950
+Wire Notes Line
+	6250 1950 6250 2350
+Text Notes 6350 2300 0    79   ~ 0
+CUT THIS LINE
 $EndSCHEMATC

Commit message: updated the repo with all latest pcb changes for the 6cell bms, 3cell bms, and for the wireless charger. Also added sensor data readme filein the same directory as the makaniu python program
Parts:
- added C24: 1uF, Capacitor_SMD:C_0402_1005Metric, symbol Device:C
- added C25: 4.7uF, Capacitor_SMD:C_0603_1608Metric, symbol Device:C
- added U7: TPS70933DBV, Package_TO_SOT_SMD:SOT-23-5, symbol Maka_BMS-rescue:TPS70933DBV-Custom
- C12: value 15nF -> 1uF; Digikey 311-1713-1-ND -> 490-10017-1-ND; LCSC (none) -> C52923; RemQ (none) -> 2
- C19: value 0.22uF -> 1uF; Digikey 490-12265-1-ND -> 490-10017-1-ND; LCSC C16772 -> C52923; RemQ 0 -> 2
- C6, C8, C9: RemQ 1 -> 2
- L2, L3: value 10uH IHLP2020 -> 10uH; footprint Inductor_SMD:L_Vishay_IHLP-2020 -> Custom:MPL-SE6040-100; Digikey 541-1093-1-ND -> 1589-MPL-SE6040-100CT-ND
- R22: LCSC C13187 -> C26974
- R25: LCSC C17765 -> C25913
- R29: value 0.06 -> 0.25; Digikey WSLC-.06CT-ND -> 311-0.25ANCT-ND
- TH2: value DNP -> 10K; Digikey 495-5814-1-ND -> 311-10.0KLRCT-ND; LCSC (none) -> C25744; RemQ (none) -> 0
Connections:
- net labels added: +3.3VP, ENDCAP_EN
- net labels removed: ~INT~
- wire segments 304 -> 317
- no-connect marks 10 -> 11
Other:
- note removed: "CUT THIS LINE"
