File: PCBs/battery_manager/Maka_BMS.sch (KiCad schematic (older format))
At the start: 88 parts, among them J8 ‎SAM16035-ND‎, J9 Molex 087340-1424, Q1 FDC645N, Q2 FDC645N, Q3 FDC645N, Q4 Si3483CDV, Q5 Si3483CDV, Q6 FDC645N, U1 AP63205, U2 TPS70933DBV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

Commit message: added a dimmensioned drawing of the Maka Niu Housing in the documentation section
Parts:
- R31: value 0.1 -> 0.05; Digikey 311-0.1ANCT-ND -> (none); LCSC C25334 -> (none); RemQ 0 -> (none)
Changed lines of the file:
@@
 P 10850 2200
 F 0 "R31" V 10750 2200 50  0000 C CNN
-F 1 "0.1" V 10850 2200 50  0000 C CNN
+F 1 "0.05" V 10850 2200 50  0000 C CNN
 F 2 "Resistor_SMD:R_1206_3216Metric_Pad1.42x1.75mm_HandSolder" V 10780 2200 50  0001 C CNN
 F 3 "~" H 10850 2200 50  0001 C CNN
-F 4 "	311-0.1ANCT-ND" H 10850 2200 50  0001 C CNN "Digikey"
-F 5 "C25334" H 10850 2200 50  0001 C CNN "LCSC"
-F 6 "0" H 10850 2200 50  0001 C CNN "RemQ"
+F 4 "" H 10850 2200 50  0001 C CNN "Digikey"
+F 5 "" H 10850 2200 50  0001 C CNN "LCSC"
+F 6 "" H 10850 2200 50  0001 C CNN "RemQ"
 	1    10850 2200
 	0    1    1    0
