File: PCBs/battery_manager_6cell/Maka_BMS.sch (KiCad schematic (older format))
At the start: 107 parts, among them J2 Conn_02x05_Odd_Even, J7 Conn_01x03, Q1 FDC645N, Q2 FDC645N, Q3 FDC645N, Q4 Si3483CDV, Q5 Si3483CDV, Q6 FDC645N, Q7 FDC645N, Q8 FDC645N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

Commit message: updates to battery managemennt wayfinder boards, and makaniu hall sensor ring and BMS
Parts:
- C1, C7: LCSC (none) -> C96446; LCSC Part Number (none) -> 0
- C10, C13: Digikey 490-7202-1-ND -> 732-7495-1-ND; LCSC (none) -> C155422; LCSC Part Number (none) -> 0
- C11, C12, C2, C25, C26, C3, C4, C5: LCSC (none) -> C155422; LCSC Part Number (none) -> 0
- C14: LCSC (none) -> C69335; LCSC Part Number (none) -> 0
- C15, C16, C17, C22, C23, C24: LCSC (none) -> C59461; LCSC Part Number (none) -> 0
- C18: Digikey (none) -> 311-3567-2-ND; LCSC (none) -> C14663; LCSC Part Number (none) -> 0
- C19: LCSC (none) -> C47129; LCSC Part Number (none) -> 0
- C20, D3, L1, L2, L3, Q1, Q2, Q3, Q4, Q5, Q6, Q7, Q8, R20, R24, R28, R29, U1, U3, U4, U5, U6, U7: LCSC part number (none) -> x
- C21: LCSC (none) -> C1538; LCSC Part Number (none) -> 0
- C27, C28, C6, C8, C9: LCSC (none) -> C52923; LCSC Part Number (none) -> 0
- D1, D2, D4: value 30V 3A -> 60V 3A; LCSC part number (none) -> x
- R1, R13, R2, R3, R34, R35, R36, R4, R41, R5, R6, R7, R9: LCSC (none) -> C11702; LCSC Part Number (none) -> 0
- R10, R15, R17, R38, R42, R44: LCSC (none) -> C25744; LCSC Part Number (none) -> 0
- R11, R12, R14, R39, R40: LCSC (none) -> C26083; LCSC Part Number (none) -> 0
- R16, R43: LCSC (none) -> C25741; LCSC Part Number (none) -> 0
- R18, R22, R45: LCSC (none) -> C25790; LCSC Part Number (none) -> 0
- R19: LCSC (none) -> C25770; LCSC Part Number (none) -> 0
- R25: LCSC (none) -> C25913; LCSC Part Number (none) -> 0
- R26, R27: LCSC (none) -> C25889; LCSC Part Number (none) -> 0
- R30: LCSC (none) -> C25876; LCSC Part Number (none) -> 0
- R31: LCSC (none) -> C25334; LCSC Part Number (none) -> 0
- R37, R8: LCSC (none) -> C127690; LCSC Part Number (none) -> 0
- TH1, TH3: Digikey P12985CT-ND -> 495-5814-1-ND; LCSC part number (none) -> x
- U2: value TPS70933DBV -> TPS70933QDBVR; LCSC part number (none) -> x/2
Other:
- note added: "Changed to 0.05ohm, \nfor 2 amp charge rate"
- note added: "limits incoming current at a 1.5Amps"

Commit message: updated the repo with all latest pcb changes for the 6cell bms, 3cell bms, and for the wireless charger. Also added sensor data readme filein the same directory as the makaniu python program
Parts:
- R23: value DNP -> 100K
- R31: value 0.1 -> 0.5; Digikey 311-0.1ANCT-ND -> (none)
Connections:
- wire segments 423 -> 427
- no-connect marks 11 -> 10
Other:
- note added: "DNP"
- note removed: "Changed to 0.05ohm, \nfor 2 amp charge rate"
