File: PCBs/battery_manager_V1.1/Maka_BMS.kicad_pcb (KiCad board)
At the start: 4 copper layers, 39 x 35.2 mm, 93 parts, among them J8 ‎SAM16035-ND‎, J9 Molex 087340-1424, Q1 FDC645N, Q2 FDC645N, Q3 FDC645N, Q4 Si3483CDV, Q5 Si3483CDV, Q6 FDC645N, U1 AP63205, U2 TPS70933DBV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

Commit message: number of PCBs for 2nd round of Maka Niu fabrication, in their state after orders made.
Parts:
- C9, R10, R12, R13, R14, R18, R20, R6: moved to B.Cu
- D3: value CRS08 -> 60V 3A; footprint Diode_SMD:D_SOD-123 -> Custom:D_SOD-123EP
- L2, L3: footprint Custom:MPL-SE6040-100 -> Custom:Inductor5x5mm
- R19: value 270K -> 390K
- R35, R36: value 10K -> DNP
- moved R14 5.80 mm to (146.3, 112.5), turned to 0 degrees
- moved R20 3.77 mm to (146.9, 113.5), turned to 180 degrees
- moved U4 2.80 mm to (147.7, 117.1), turned to 90 degrees
- moved R10 0.43 mm to (139.6, 101.1)
- moved L2 0.27 mm to (166.3, 109.4)
- moved R6 0.20 mm to (144.6, 88.8), turned to 180 degrees
- moved L1 0.20 mm to (151.9, 117.5)
Connections:
- net ~DELAYED_OFF~ renamed ~{DELAYED_OFF}
- net ~SHT_DWN_SIG~ renamed ~{SHT_DWN_SIG}
- net ~TS_EOC~ renamed ~{TS_EOC}
- J9 pad 11: Net-(J9-Pad11) -> unconnected-(J9-Pad11)
- J9 pad 3: Net-(J9-Pad3) -> unconnected-(J9-Pad3)
- J9 pad 9: Net-(J9-Pad9) -> unconnected-(J9-Pad9)
- U2 pad 3: Net-(U2-Pad3) -> unconnected-(U2-Pad3)
- U3 pad 15: Net-(U3-Pad15) -> unconnected-(U3-Pad15)
- U3 pad 21: Net-(U3-Pad21) -> unconnected-(U3-Pad21)
- U5 pad 12: Net-(U5-Pad12) -> unconnected-(U5-Pad12)
- U5 pad 13: Net-(U5-Pad13) -> unconnected-(U5-Pad13)
- U5 pad 16: Net-(U5-Pad16) -> unconnected-(U5-Pad16)
- U5 pad 3: Net-(U5-Pad3) -> unconnected-(U5-Pad3)
- U5 pad 5: Net-(U5-Pad5) -> unconnected-(U5-Pad5)
- U5 pad 8: Net-(U5-Pad8) -> unconnected-(U5-Pad8)
Routing:
- net +5V: track 50.1 -> 37.8 mm, vias 5 -> 4
- net Net-(R19-Pad2): track 2.16 -> 8.88 mm, vias 0 -> 2
- net ~{SHT_DWN_SIG}: track 18.0 -> 13.6 mm, vias 3 -> 2
- net +12V: track 37.4 -> 41.8 mm
- net Net-(C21-Pad2): track 6.33 -> 9.27 mm
- net +3V3: track 62.5 -> 65.3 mm
- net Earth: track 102.4 -> 101.0 mm, vias 22 -> 23
- net ENDCAP_EN: track 18.4 -> 17.1 mm
- net ~{DELAYED_OFF}: track 50.3 -> 51.6 mm, vias 2 -> 1
- net Net-(Q1-Pad2): track 1.72 -> 2.76 mm, vias 0 -> 1
- net Net-(R14-Pad2): track 2.58 -> 3.54 mm, vias 0 -> 1
- net /BATT_OUT: track 46.8 -> 45.9 mm
- net Net-(Q2-Pad2): track 3.27 -> 2.48 mm
- net Net-(R21-Pad2): track 10.6 -> 11.3 mm
- net SDA: track 51.4 -> 50.8 mm
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Other:
- net class 1.5A_Amp removed
- net class 2.2A_Power removed
- net class Default removed
