File: PCBs/battery_manager_V1.1/Maka_BMS.sch (KiCad schematic (older format))
At the start: 93 parts, among them J8 ‎SAM16035-ND‎, J9 Molex 087340-1424, Q1 FDC645N, Q2 FDC645N, Q3 FDC645N, Q4 Si3483CDV, Q5 Si3483CDV, Q6 FDC645N, U1 AP63205, U2 TPS70933DBV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

Commit message: number of PCBs for 2nd round of Maka Niu fabrication, in their state after orders made.
Parts:
- R35, R36: value 10K -> DNP; Digikey 311-10.0KLRCT-ND -> (none); LCSC C25744 -> (none); RemQ 2 -> (none)
Changed lines of the file:
@@
 Text Label 7900 6050 1    79   ~ 0
 Batt_Analog
-Wire Wire Line
-	8150 5650 8000 5650
-Connection ~ 8150 5650
-Wire Wire Line
-	9100 5250 8150 5250
-Connection ~ 9100 5250
-Wire Wire Line
-	8150 5250 8150 5650
-Wire Wire Line
-	9500 5250 9100 5250
-$Comp
-L Device:R R36
-U 1 1 632E60A4
-P 9500 5400
-F 0 "R36" H 9430 5354 50  0000 R CNN
-F 1 "10K" H 9430 5445 50  0000 R CNN
-F 2 "Resistor_SMD:R_0402_1005Metric" V 9430 5400 50  0001 C CNN
-F 3 "~" H 9500 5400 50  0001 C CNN
-F 4 "	311-10.0KLRCT-ND" H 9500 5400 50  0001 C CNN "Digikey"
-F 5 "C25744" H 9500 5400 50  0001 C CNN "LCSC"
-F 6 "2" H 9500 5400 50  0001 C CNN "RemQ"
-	1    9500 5400
-	-1   0    0    1
-$EndComp
-$Comp
-L Device:R R35
-U 1 1 632E565B
-P 9100 5400
-F 0 "R35" H 9030 5354 50  0000 R CNN
-F 1 "10K" H 9030 5445 50  0000 R CNN
-F 2 "Resistor_SMD:R_0402_1005Metric" V 9030 5400 50  0001 C CNN
-F 3 "~" H 9100 5400 50  0001 C CNN
-F 4 "	311-10.0KLRCT-ND" H 9100 5400 50  0001 C CNN "Digikey"
-F 5 "C25744" H 9100 5400 50  0001 C CNN "LCSC"
-F 6 "2" H 9100 5400 50  0001 C CNN "RemQ"
-	1    9100 5400
-	-1   0    0    1
-$EndComp
-Wire Wire Line
-	9100 5950 9000 5950
-Connection ~ 9100 5950
-Wire Wire Line
-	9500 6100 9500 5550
-Wire Wire Line
-	9100 6100 9500 6100
-Wire Wire Line
-	9100 5950 9100 6100
-Wire Wire Line
-	9100 5750 9200 5750
-Connection ~ 9100 5750
-Wire Wire Line
-	9100 5750 9100 5550
-Wire Wire Line
-	9000 5750 9100 5750
 Text Notes 9800 6300 0    79   ~ 0
 Battery voltage ADC
@@
 Wire Wire Line
 	8000 5650 8000 5600
-Wire Wire Line
-	8200 5650 8150 5650
 $Comp
 L power:Earth #PWR045
@@
 Wire Wire Line
 	8200 6050 8000 6050
-Wire Wire Line
-	9200 5950 9100 5950
 Text GLabel 9200 5750 2    50   Output ~ 0
 SCL
@@
 Wire Wire Line
 	8000 6050 8000 6200
+Wire Wire Line
+	8200 5650 8150 5650
+Wire Wire Line
+	8150 5650 8000 5650
+Connection ~ 8150 5650
+Wire Wire Line
+	8150 5250 8150 5650
+Wire Wire Line
+	9200 5950 9100 5950
+Wire Wire Line
+	9100 5950 9000 5950
+Connection ~ 9100 5950
+Wire Wire Line
+	9100 5950 9100 6100
+Wire Wire Line
+	9100 6100 9500 6100
+Wire Wire Line
+	9500 6100 9500 5550
+Wire Wire Line
+	9000 5750 9100 5750
+Wire Wire Line
+	9100 5750 9200 5750
+Connection ~ 9100 5750
+Wire Wire Line
+	9100 5750 9100 5550
+Wire Wire Line
+	9500 5250 9100 5250
+Wire Wire Line
+	9100 5250 8150 5250
+Connection ~ 9100 5250
+$Comp
+L Device:R R35
+U 1 1 632E565B
+P 9100 5400
+F 0 "R35" H 9030 5354 50  0000 R CNN
+F 1 "DNP" H 9030 5445 50  0000 R CNN
+F 2 "Resistor_SMD:R_0402_1005Metric" V 9030 5400 50  0001 C CNN
+F 3 "~" H 9100 5400 50  0001 C CNN
+F 4 "" H 9100 5400 50  0001 C CNN "Digikey"
+F 5 "" H 9100 5400 50  0001 C CNN "LCSC"
+F 6 "" H 9100 5400 50  0001 C CNN "RemQ"
+	1    9100 5400
+	-1   0    0    1
+$EndComp
+$Comp
+L Device:R R36
+U 1 1 632E60A4
+P 9500 5400
+F 0 "R36" H 9430 5354 50  0000 R CNN
+F 1 "DNP" H 9430 5445 50  0000 R CNN
+F 2 "Resistor_SMD:R_0402_1005Metric" V 9430 5400 50  0001 C CNN
+F 3 "~" H 9500 5400 50  0001 C CNN
+F 4 "" H 9500 5400 50  0001 C CNN "Digikey"
+F 5 "" H 9500 5400 50  0001 C CNN "LCSC"
+F 6 "" H 9500 5400 50  0001 C CNN "RemQ"
+	1    9500 5400
+	-1   0    0    1
+$EndComp
 $EndSCHEMATC
