File: PCBs/hall_ring_V2/Hall_ring.kicad_pcb (KiCad board)
At the start: 2 copper layers, 38.5 x 37 mm, 18 parts, among them J1 T1M-06-X-DV, U1 DRV5053_LPG, U2 DRV5053_LPG, U3 DRV5053_LPG, U4 DRV5053_LPG, U5 DRV5053_LPG, U6 DRV5053_LPG, U7 DRV5053_LPG

Commit message: number of PCBs for 2nd round of Maka Niu fabrication, in their state after orders made.
Parts:
- U1, U2, U3, U4, U5, U6, U7: footprint Package_TO_SOT_THT:TO-92Flat -> Custom:TO-92Flat
Routing:
- net VCC: track 98.7 -> 97.5 mm
- net Net-(D1-Pad1): track 3.03 -> 2.18 mm
Other:
- net class Default removed
